Commit message: Updated with Pose Editor
Added the ability to create a Pose and drop it into the timeline, or save it to a Library with an image automatically created.

File: ServoAnimator/Models/johnny5_head.urdf (robot description, URDF)
Before this commit: robot servo_animator_head, 51 links, 50 joints
Joints:
- joint Microphone_RaiseLower: origin xyz=0.011362 -0.083909 0.059267 rpy=0 0 0 -> xyz=0.000362 -0.083909 0.056267 rpy=0 0 0

Commit message: Numerous UI updates, new looping sequences
Added looping Sequences
Updated UI and memory of UI settings.
Added auto save and recovery

File: ServoAnimator/Models/johnny5_head.urdf (robot description, URDF)
Before this commit: robot servo_animator_head, 51 links, 50 joints
Joints:
- joint MFR_UpDown: limit lower=0.000000 upper=0.052917 effort=5 velocity=0.2 -> lower=0.022429906542056 upper=0.065105386416862 effort=5 velocity=0.2
- joint Microphone_RaiseLower: limit lower=0.000000 upper=0.011430 effort=5 velocity=0.15 -> lower=0.000000 upper=0.010000 effort=5 velocity=0.15

Commit message: Update Animation Editor controllers, calibrated motion, API, and deployment 1.26.5

File: ServoAnimator/Models/johnny5_head.urdf (robot description, URDF)
Before this commit: robot servo_animator_head, 51 links, 50 joints
Links:
- link head_link: geometry collision mesh filename=Meshes/RearCover/rear_cover_collision_full.stl scale=0.001000 0.001000 0.001000; collision mesh filename=Meshes/SimpleMouth/lip_led_00_collision_full.stl scale=0.001000 0.001000 0.001000
- link left_bottom_flap_link: geometry collision mesh filename=Meshes/SimplifiedHead2/lower_left_flap_panel_collision_full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 scale=0.001000 0.001000 0.001000; visual mesh filename=Meshes/SimplifiedHead2/lower_left_arm_hardware.stl scale=0.001000 0.001000 0.001000
- link left_eye_pop_link: geometry collision mesh filename=Meshes/EyeMechanism/eye_fixed_cad1ee_rest_without_gimbal_sp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 scale=0.001000 0.001000 0.001000; collision mesh filename=Meshes/EyeMechanism/eye_fixed_f6f6f3_collision_full.stl scale=0.001000 0.001000 0.001000
- link left_eye_v_link: geometry collision mesh filename=Meshes/EyeMechanism/eye_gimbal_a0a0a0_collision_full.stl scale=0.001000 0.001000 0.001000; visual mesh filename=Meshes/EyeMechanism/eye_gimbal_a0a0a0.stl scale=0.001000 0.001000 0.001000
- link left_eye_vent_fin1_link: geometry collision mesh filename=Meshes/SimplifiedHead2/vent_left_fin1_collision_full.stl scale=0.001000 0.001000 0.001000; visual mesh filename=Meshes/SimplifiedHead2/vent_left_fin1.stl scale=0.001000 0.001000 0.001000
- link left_eye_vent_fin2_link: geometry collision mesh filename=Meshes/SimplifiedHead2/vent_left_fin2_collision_full.stl scale=0.001000 0.001000 0.001000; visual mesh filename=Meshes/SimplifiedHead2/vent_left_fin2.stl scale=0.001000 0.001000 0.001000
- link left_eye_vent_fin3_link: geometry collision mesh filename=Meshes/SimplifiedHead2/vent_left_fin3_collision_full.stl scale=0.001000 0.001000 0.001000; visual mesh filename=Meshes/SimplifiedHead2/vent_left_fin3.stl scale=0.001000 0.001000 0.001000
- link left_eye_vent_fin4_link: geometry collision mesh filename=Meshes/SimplifiedHead2/vent_left_fin4_collision_full.stl scale=0.001000 0.001000 0.001000; visual mesh filename=Meshes/SimplifiedHead2/vent_left_fin4.stl scale=0.001000 0.001000 0.001000
- link left_eye_vent_fin5_link: geometry collision mesh filename=Meshes/SimplifiedHead2/vent_left_fin5_collision_full.stl scale=0.001000 0.001000 0.001000; visual mesh filename=Meshes/SimplifiedHead2/vent_left_fin5.stl scale=0.001000 0.001000 0.001000
- link left_eye_vent_link: geometry collision mesh filename=Meshes/SimplifiedHead2/vent_left_drive_collision_full.stl scale=0.001000 0.001000 0.001000; visual mesh filename=Meshes/SimplifiedHead2/vent_left_drive.stl scale=0.001000 0.001000 0.001000
- link left_pupil_link: geometry collision cylinder length=0.003175 radius=0.022860; collision mesh filename=Meshes/EyeMechanism/iris_gold_continuous_collision_full.stl scale=0.001 0.001 0.001
- link left_top_ball_link: geometry collision mesh filename=Meshes/NeckAssembly/left_top_ball_collision_full.stl scale=0.001000 0.001000 0.001000; visual mesh filename=Meshes/NeckAssembly/left_top_ball.stl scale=0.001000 0.001000 0.001000
- link left_top_flap_link: geometry collision mesh filename=Meshes/SimplifiedHead2/upper_left_flap_panel_collision_full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 scale=0.001000 0.001000 0.001000; visual mesh filename=Meshes/SimplifiedHead2/upper_left_flap_panel.stl scale=0.001000 0.001000 0.001000
- link mfr_rotate_link: geometry collision mesh filename=Meshes/HeadTopCAD/MFRC_404040_collision_full.stl scale=0.001000 0.001000 0.001000; collision mesh filename=Meshes/HeadTopCAD/MFRC_97a3da_collision_full.stl scale=0.001000 0.001000 0.001000
- link microphone_link: geometry collision mesh filename=Meshes/HeadTopCAD/Microphone_97a3da_collision_full.stl scale=0.001000 0.001000 0.001000; collision mesh filename=Meshes/HeadTopCAD/Microphone_b5afa6_collision_full.stl scale=0.001000 0.001000 0.001000
- link nose_basket_link: geometry collision mesh filename=Meshes/SimplifiedHead2/nose_basket_collision_full.stl scale=0.001000 0.001000 0.001000; visual mesh filename=Meshes/SimplifiedHead2/nose_basket.stl scale=0.001000 0.001000 0.001000
- link nose_body_link: geometry collision mesh filename=Meshes/SimplifiedHead2/nose_body_collision_full.stl scale=0.001000 0.001000 0.001000; visual mesh filename=Meshes/SimplifiedHead2/nose_body.stl scale=0.001000 0.001000 0.001000
- link right_bottom_flap_link: geometry collision mesh filename=Meshes/SimplifiedHead2/lower_right_flap_panel_collision_ful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 scale=0.001000 0.001000 0.001000; visual mesh filename=Meshes/SimplifiedHead2/lower_right_arm_hardware.stl scale=0.001000 0.001000 0.001000
- link right_eye_pop_link: geometry collision mesh filename=Meshes/EyeMechanism/eye_fixed_cad1ee_rest_without_gimbal_sp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 scale=0.001000 0.001000 0.001000; collision mesh filename=Meshes/EyeMechanism/eye_fixed_f6f6f3_collision_full.stl scale=0.001000 0.001000 0.001000
- link right_eye_v_link: geometry collision mesh filename=Meshes/EyeMechanism/eye_gimbal_a0a0a0_collision_full.stl scale=0.001000 0.001000 0.001000; visual mesh filename=Meshes/EyeMechanism/eye_gimbal_a0a0a0.stl scale=0.001000 0.001000 0.001000
- link right_eye_vent_fin1_link: geometry collision mesh filename=Meshes/SimplifiedHead2/vent_right_fin1_collision_full.stl scale=0.001000 0.001000 0.001000; visual mesh filename=Meshes/SimplifiedHead2/vent_right_fin1.stl scale=0.001000 0.001000 0.001000
- link right_eye_vent_fin2_link: geometry collision mesh filename=Meshes/SimplifiedHead2/vent_right_fin2_collision_full.stl scale=0.001000 0.001000 0.001000; visual mesh filename=Meshes/SimplifiedHead2/vent_right_fin2.stl scale=0.001000 0.001000 0.001000
- link right_eye_vent_fin3_link: geometry collision mesh filename=Meshes/SimplifiedHead2/vent_right_fin3_collision_full.stl scale=0.001000 0.001000 0.001000; visual mesh filename=Meshes/SimplifiedHead2/vent_right_fin3.stl scale=0.001000 0.001000 0.001000
- link right_eye_vent_fin4_link: geometry collision mesh filename=Meshes/SimplifiedHead2/vent_right_fin4_collision_full.stl scale=0.001000 0.001000 0.001000; visual mesh filename=Meshes/SimplifiedHead2/vent_right_fin4.stl scale=0.001000 0.001000 0.001000
- link right_eye_vent_fin5_link: geometry collision mesh filename=Meshes/SimplifiedHead2/vent_right_fin5_collision_full.stl scale=0.001000 0.001000 0.001000; visual mesh filename=Meshes/SimplifiedHead2/vent_right_fin5.stl scale=0.001000 0.001000 0.001000
- link right_eye_vent_link: geometry collision mesh filename=Meshes/SimplifiedHead2/vent_right_drive_collision_full.stl scale=0.001000 0.001000 0.001000; visual mesh filename=Meshes/SimplifiedHead2/vent_right_drive.stl scale=0.001000 0.001000 0.001000
- link right_pupil_link: geometry collision cylinder length=0.003175 radius=0.022860; collision mesh filename=Meshes/EyeMechanism/iris_gold_continuous_collision_full.stl scale=0.001 0.001 0.001
- link right_top_ball_link: geometry collision mesh filename=Meshes/NeckAssembly/right_top_ball_collision_full.stl scale=0.001000 0.001000 0.001000; visual mesh filename=Meshes/NeckAssembly/right_top_ball.stl scale=0.001000 0.001000 0.001000
- link right_top_flap_link: geometry collision mesh filename=Meshes/SimplifiedHead2/upper_right_flap_panel_collision_ful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 scale=0.001000 0.001000 0.001000; visual mesh filename=Meshes/SimplifiedHead2/upper_right_flap_panel.stl scale=0.001000 0.001000 0.001000
- link whip_fold_link: geometry collision mesh filename=Meshes/HeadTopCAD/WhipAntenna_upper_knob_collision_full.stl scale=0.001 0.001 0.001; collision mesh filename=Meshes/HeadTopCAD/WhipAntenna_upper_linkage_collision_full.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 scale=0.001 0.001 0.001
- link whip_rotate_link: geometry collision mesh filename=Meshes/HeadTopCAD/WhipAntenna_hinge_pin_collision_full.stl scale=0.001 0.001 0.001; collision mesh filename=Meshes/HeadTopCAD/WhipAntenna_lower_linkage_collision_full.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 scale=0.001 0.001 0.001
